Commit message: modidy link and joint name

File: zx120_description/urdf/zx120.xacro (robot description, xacro)
@@ -4,13 +4,13 @@
 	<xacro:include filename="$(find zx120_description)/urdf/zx120.gazebo" />
 	<!-- Import Rviz colors -->
-	<xacro:include filename="$(find zx120_description)/urdf/materials.xacro" />
-	<!-- Used for fixing robot to Gazebo 'base_link' -->
-	<link name="world"/>
-	<joint name="fixed" type="fixed">
-		<parent link="world"/>
-		<child link="link1"/>
-	</joint>
+	<!-- <xacro:include filename="$(find zx120_description)/urdf/materials.xacro" /> -->
 	<!-- Base Link -->
-	<link name="link1">
+	<link name="base_link"/>
+	<joint name="base_joint" type="fixed">
+		<parent link="base_link"/>
+		<child link="track_link"/>
+	</joint>
+	<!-- Base Link -->
+	<link name="track_link">
 		<visual>
 			<geometry>
@@ -32,11 +32,11 @@
 	</link>
 	<!-- body axis -->
-	<joint name="joint1" type="continuous">
+	<joint name="body_joint" type="continuous">
 		<origin xyz="0 0 1"/>
 		<axis xyz="0 0 2"/>
-		<parent link="link1"/>
-		<child link="link2"/>
-	</joint>
-	<link name="link2">
+		<parent link="track_link"/>
+		<child link="body_link"/>
+	</joint>
+	<link name="body_link">
 		<visual>
 			<origin xyz="0 0 0"/>
@@ -60,23 +60,23 @@
 	</link>
 	<!-- boom axis -->
-	<joint name="joint2" type="revolute">
+	<joint name="boom_joint" type="revolute">
 		<origin xyz="0.15433 -0.16443 0.31327"/>
 		<axis xyz="0 1 0"/>
-		<parent link="link2"/>
-		<child link="link3"/>
+		<parent link="body_link"/>
+		<child link="boom_link"/>
 		<limit lower="${radians(-70)}" upper="${radians(30)}" effort="500" velocity="6.159937255"/>
 	</joint>
-	<joint name="joint5" type="continuous">
+	<joint name="boom_cylinder_head_joint" type="continuous">
 		<origin xyz="0.556105 -0.164428 0.032962"/>
 		<axis xyz="0 1 0"/>
-		<parent link="link2"/>
-		<child link="link6"/>
-		<mimic joint="joint2" multiplier="${60/70}"/>
-	</joint>
-	<gazebo>
-		<plugin name="joint5_mimic_joint_plugin"
-				filename="libroboticsgroup_upatras_gazebo_mimic_joint_plugin.so">
-			<joint>joint2</joint>
-			<mimicJoint>joint5</mimicJoint>
+		<parent link="body_link"/>
+		<child link="boom_cylinder_head_link"/>
+		<mimic joint="boom_joint" multiplier="${60/70}"/>
+	</joint>
+	<gazebo>
+		<plugin name="boom_cylinder_head_joint_mimic_joint_plugin"
+				filename="libroboticsgroup_upatras_gazebo_mimic_joint_plugin.so">
+			<joint>boom_joint</joint>
+			<mimicJoint>boom_cylinder_head_joint</mimicJoint>
 			<multiplier>${60/70}</multiplier>
 			<offset>0</offset>
@@ -84,17 +84,17 @@
 		</plugin>
 	</gazebo>
-	<joint name="joint6" type="prismatic">
+	<joint name="boom_cylinder_rod_joint" type="prismatic">
 		<origin xyz="0 0 0"/>
 		<axis xyz="0.802033 0 1.847495"/>
-		<parent link="link6"/>
-		<child link="link7"/>
+		<parent link="boom_cylinder_head_link"/>
+		<child link="boom_cylinder_rod_link"/>
 		<limit lower="-2" upper="2" effort="500" velocity="6.159937255"/>
-		<mimic joint="joint2" multiplier="${0.39/-1.22}"/>
-	</joint>
-	<gazebo>
-		<plugin name="joint6_mimic_joint_plugin"
-				filename="libroboticsgroup_upatras_gazebo_mimic_joint_plugin.so">
-			<joint>joint2</joint>
-			<mimicJoint>joint6</mimicJoint>
+		<mimic joint="boom_joint" multiplier="${0.39/-1.22}"/>
+	</joint>
+	<gazebo>
+		<plugin name="boom_cylinder_rod_joint_mimic_joint_plugin"
+				filename="libroboticsgroup_upatras_gazebo_mimic_joint_plugin.so">
+			<joint>boom_joint</joint>
+			<mimicJoint>boom_cylinder_rod_joint</mimicJoint>
 			<multiplier>${0.39/-1.22}</multiplier>
 			<offset>0</offset>
@@ -102,23 +102,23 @@
 		</plugin>
 	</gazebo>
-	<joint name="joint7" type="fixed">
+	<joint name="arm_cylinder_head_joint" type="fixed">
 		<origin xyz="2.053030 0 1.991444"/>
 		<axis xyz="0 1 0"/>
-		<parent link="link3"/>
-		<child link="link8"/>
-	</joint>
-	<joint name="joint8" type="prismatic">
+		<parent link="boom_link"/>
+		<child link="arm_cylinder_head_link"/>
+	</joint>
+	<joint name="arm_cylinder_rod_joint" type="prismatic">
 		<origin xyz="0 0 0"/>
 		<axis xyz="2.36471 0 0"/>
-		<parent link="link8"/>
-		<child link="link9"/>
+		<parent link="arm_cylinder_head_link"/>
+		<child link="arm_cylinder_rod_link"/>
 		<limit lower="-2" upper="2" effort="500" velocity="6.159937255"/>
-		<mimic joint="joint3" multiplier="${0.4/radians(50)}"/>
-	</joint>
-	<gazebo>
-		<plugin name="joint8_mimic_joint_plugin"
-				filename="libroboticsgroup_upatras_gazebo_mimic_joint_plugin.so">
-			<joint>joint3</joint>
-			<mimicJoint>joint8</mimicJoint>
+		<mimic joint="arm_joint" multiplier="${0.4/radians(50)}"/>
+	</joint>
+	<gazebo>
+		<plugin name="arm_cylinder_rod_joint_mimic_joint_plugin"
+				filename="libroboticsgroup_upatras_gazebo_mimic_joint_plugin.so">
+			<joint>arm_joint</joint>
+			<mimicJoint>arm_cylinder_rod_joint</mimicJoint>
 			<multiplier>${0.4/radians(50)}</multiplier>
 			<offset>0</offset>
@@ -126,23 +126,23 @@
 		</plugin>
 	</gazebo>
-	<joint name="joint9" type="fixed">
+	<joint name="bucket_cylinder_head_joint" type="fixed">
 		<origin xyz="0.605825 0 -0.364793"/>
 		<axis xyz="0 1 0"/>
-		<parent link="link4"/>
-		<child link="link10"/>
-	</joint>
-	<joint name="joint10" type="prismatic">
+		<parent link="arm_link"/>
+		<child link="bucket_cylinder_head_link"/>
+	</joint>
+	<joint name="bucket_cylinder_rod_joint" type="prismatic">
 		<origin xyz="0 0 0"/>
 		<axis xyz="-0.021529 0 -2.207579"/>
-		<parent link="link10"/>
-		<child link="link11"/>
+		<parent link="bucket_cylinder_head_link"/>
+		<child link="bucket_cylinder_rod_link"/>
 		<limit lower="-2" upper="2" effort="500" velocity="6.159937255"/>
-		<mimic joint="joint4" multiplier="${-0.9/-2.79}"/>
-	</joint>
-	<gazebo>
-		<plugin name="joint10_mimic_joint_plugin"
-				filename="libroboticsgroup_upatras_gazebo_mimic_joint_plugin.so">
-			<joint>joint4</joint>
-			<mimicJoint>joint10</mimicJoint>
+		<mimic joint="bucket_joint" multiplier="${-0.9/-2.79}"/>
+	</joint>
+	<gazebo>
+		<plugin name="bucket_cylinder_rod_joint_mimic_joint_plugin"
+				filename="libroboticsgroup_upatras_gazebo_mimic_joint_plugin.so">
+			<joint>bucket_joint</joint>
+			<mimicJoint>bucket_cylinder_rod_joint</mimicJoint>
 			<multiplier>${-0.9/-2.79}</multiplier>
 			<offset>0</offset>
@@ -150,16 +150,16 @@
 		</plugin>
 	</gazebo>
-	<joint name="joint11" type="continuous">
+	<joint name="bucket_b_joint" type="continuous">
 		<origin xyz="0.330489 0 -2.150643"/>
 		<axis xyz="0 1 0"/>
-		<parent link="link4"/>
-		<child link="link12"/>
-		<mimic joint="joint4" multiplier="${120/160}"/>
-	</joint>
-	<gazebo>
-		<plugin name="joint11_mimic_joint_plugin"
-				filename="libroboticsgroup_upatras_gazebo_mimic_joint_plugin.so">
-			<joint>joint4</joint>
-			<mimicJoint>joint11</mimicJoint>
+		<parent link="arm_link"/>
+		<child link="bucket_b_link"/>
+		<mimic joint="bucket_joint" multiplier="${120/160}"/>
+	</joint>
+	<gazebo>
+		<plugin name="bucket_b_joint_mimic_joint_plugin"
+				filename="libroboticsgroup_upatras_gazebo_mimic_joint_plugin.so">
+			<joint>bucket_joint</joint>
+			<mimicJoint>bucket_b_joint</mimicJoint>
 			<multiplier>${120/160}</multiplier>
 			<offset>0</offset>
@@ -167,16 +167,16 @@
 		</plugin>
 	</gazebo>
-	<joint name="joint12" type="continuous">
+	<joint name="bucket_a_joint" type="continuous">
 		<origin xyz="-0.182145 0 -0.315076"/>
 		<axis xyz="0 1 0"/>
-		<parent link="link5"/>
-		<child link="link13"/>
-		<mimic joint="joint4" multiplier="${-92/160}"/>
-	</joint>
-	<gazebo>
-		<plugin name="joint12_mimic_joint_plugin"
-				filename="libroboticsgroup_upatras_gazebo_mimic_joint_plugin.so">
-			<joint>joint4</joint>
-			<mimicJoint>joint12</mimicJoint>
+		<parent link="bucket_link"/>
+		<child link="bucket_a_link"/>
+		<mimic joint="bucket_joint" multiplier="${-92/160}"/>
+	</joint>
+	<gazebo>
+		<plugin name="bucket_a_joint_mimic_joint_plugin"
+				filename="libroboticsgroup_upatras_gazebo_mimic_joint_plugin.so">
+			<joint>bucket_joint</joint>
+			<mimicJoint>bucket_a_joint</mimicJoint>
 			<multiplier>${-92/160}</multiplier>
 			<offset>0</offset>
@@ -184,5 +184,5 @@
 		</plugin>
 	</gazebo>
-	<link name="link3">
+	<link name="boom_link">
 		<visual>
 			<origin xyz="0 0 0"/>
@@ -205,12 +205,12 @@
 		</inertial>
 	</link>
-	<joint name="joint3" type="revolute">
+	<joint name="arm_joint" type="revolute">
 		<origin xyz="4.2241 0 1.7311"/>
 		<axis xyz="0 1 0"/>
-		<parent link="link3"/>
-		<child link="link4"/>
+		<parent link="boom_link"/>
+		<child link="arm_link"/>
 		<limit lower="${radians(-70)}" upper="${radians(50)}" effort="500" velocity="6.159937255"/>
 	</joint>
-	<link name="link4">
+	<link name="arm_link">
 		<visual>
 			<origin xyz="0 0 0"/>
@@ -234,12 +234,12 @@
 	</link>
 	<!-- bucket axis -->
-	<joint name="joint4" type="revolute">
+	<joint name="bucket_joint" type="revolute">
 		<origin xyz="0.35383 0 -2.4712"/>
 		<axis xyz="0 1 0"/>
-		<parent link="link4"/>
-		<child link="link5"/>
+		<parent link="arm_link"/>
+		<child link="bucket_link"/>
 		<limit lower="${radians(-160)}" upper="0" effort="500" velocity="6.159937255"/>
 	</joint>
-	<link name="link5">
+	<link name="bucket_link">
 		<visual>
 			<origin xyz="0 0 0"/>
@@ -262,5 +262,5 @@
 		</inertial>
 	</link>
-	<link name="link6">
+	<link name="boom_cylinder_head_link">
 		<visual>
 			<origin xyz="0 0 0"/>
@@ -283,5 +283,5 @@
 		</inertial>
 	</link>
-	<link name="link7">
+	<link name="boom_cylinder_rod_link">
 		<visual>
 			<origin xyz="0 0 0"/>
@@ -304,5 +304,5 @@
 		</inertial>
 	</link>
-	<link name="link8">
+	<link name="arm_cylinder_head_link">
 		<visual>
 			<origin xyz="0 0 0"/>
@@ -325,5 +325,5 @@
 		</inertial>
 	</link>
-	<link name="link9">
+	<link name="arm_cylinder_rod_link">
 		<visual>
 			<origin xyz="0 0 0"/>
@@ -346,5 +346,5 @@
 		</inertial>
 	</link>
-	<link name="link10">
+	<link name="bucket_cylinder_head_link">
 		<visual>
 			<origin xyz="0 0 0"/>
@@ -367,5 +367,5 @@
 		</inertial>
 	</link>
-	<link name="link11">
+	<link name="bucket_cylinder_rod_link">
 		<visual>
 			<origin xyz="0 0 0"/>
@@ -388,5 +388,5 @@
 		</inertial>
 	</link>
-	<link name="link12">
+	<link name="bucket_b_link">
 		<visual>
 			<origin xyz="0 0 0"/>
@@ -409,5 +409,5 @@
 		</inertial>
 	</link>
-	<link name="link13">
+	<link name="bucket_a_link">
 		<visual>
 			<origin xyz="0 0 0"/>
@@ -432,5 +432,5 @@
 	<transmission name="tran1">
 		<type>transmission_interface/SimpleTransmission</type>
-		<joint name="joint1">
+		<joint name="body_joint">
 			<hardwareInterface>hardware_interface/EffortJointInterface</hardwareInterface>
 		</joint>
@@ -442,5 +442,5 @@
 	<transmission name="tran2">
 		<type>transmission_interface/SimpleTransmission</type>
-		<joint name="joint2">
+		<joint name="boom_joint">
 			<hardwareInterface>hardware_interface/EffortJointInterface</hardwareInterface>
 		</joint>
@@ -452,5 +452,5 @@
 	<transmission name="tran3">
 		<type>transmission_interface/SimpleTransmission</type>
-		<joint name="joint3">
+		<joint name="arm_joint">
 			<hardwareInterface>hardware_interface/EffortJointInterface</hardwareInterface>
 		</joint>
@@ -462,5 +462,5 @@
 	<transmission name="tran4">
 		<type>transmission_interface/SimpleTransmission</type>
-		<joint name="joint4">
+		<joint name="bucket_joint">
 			<hardwareInterface>hardware_interface/EffortJointInterface</hardwareInterface>
 		</joint>

Commit message: modify swing(rotator) joint name

File: zx120_description/urdf/zx120.xacro (robot description, xacro)
@@ -32,5 +32,5 @@
 	</link>
 	<!-- body axis -->
-	<joint name="body_joint" type="continuous">
+	<joint name="swing_joint" type="continuous">
 		<origin xyz="0 0 1"/>
 		<axis xyz="0 0 2"/>
@@ -432,6 +432,5 @@
 	<transmission name="tran1">
 		<type>transmission_interface/SimpleTransmission</type>
-		<joint name="body_joint">
-			<hardwareInterface>hardware_interface/EffortJointInterface</hardwareInterface>
+		<joint name="swing_joint">
 		</joint>
 		<actuator name="motor1">

Commit message: add bucket end link and joint

File: zx120_description/urdf/zx120.xacro (robot description, xacro)
@@ -262,172 +262,30 @@
 		</inertial>
 	</link>
-	<link name="boom_cylinder_head_link">
-		<visual>
-			<origin xyz="0 0 0"/>
-			<geometry>
-				<mesh filename="package://zx120_description/meshes/zx120-boom-cyl1.dae"/>
-			</geometry>
-		</visual>
-		<collision>
-			<origin xyz="0 0 0"/>
-			<geometry>
-				<mesh filename="package://zx120_description/meshes/zx120-boom-cyl1.dae"/>
-			</geometry>
-		</collision>
-		<inertial>
-			<origin xyz="0.241225 0.000050 0.577034" rpy="0 0 0"/>
-			<mass value="0.03"/>
-			<inertia ixx="1.0" ixy="0.0" ixz="0.0"
-								iyy="1.0" iyz="0.0"
-											izz="1.0"/>
-		</inertial>
-	</link>
-	<link name="boom_cylinder_rod_link">
-		<visual>
-			<origin xyz="0 0 0"/>
-			<geometry>
-				<mesh filename="package://zx120_description/meshes/zx120-boom-cyl2.dae"/>
-			</geometry>
-		</visual>
-		<collision>
-			<origin xyz="0 0 0"/>
-			<geometry>
-				<mesh filename="package://zx120_description/meshes/zx120-boom-cyl2.dae"/>
-			</geometry>
-		</collision>
-		<inertial>
-			<origin xyz="0.558044 0.000050 1.286359" rpy="0 0 0"/>
-			<mass value="0.03"/>
-			<inertia ixx="1.0" ixy="0.0" ixz="0.0"
-								iyy="1.0" iyz="0.0"
-											izz="1.0"/>
-		</inertial>
-	</link>
-	<link name="arm_cylinder_head_link">
-		<visual>
-			<origin xyz="0 0 0"/>
-			<geometry>
-				<mesh filename="package://zx120_description/meshes/zx120-arm-cyl1.dae"/>
-			</geometry>
-		</visual>
-		<collision>
-			<origin xyz="0 0 0"/>
-			<geometry>
-				<mesh filename="package://zx120_description/meshes/zx120-arm-cyl1.dae"/>
-			</geometry>
-		</collision>
-		<inertial>
-			<origin xyz="0.696672 0.000026 -0.000065" rpy="0 0 0"/>
-			<mass value="0.03"/>
-			<inertia ixx="1.0" ixy="0.0" ixz="0.0"
-								iyy="1.0" iyz="0.0"
-											izz="1.0"/>
-		</inertial>
-	</link>
-	<link name="arm_cylinder_rod_link">
-		<visual>
-			<origin xyz="0 0 0"/>
-			<geometry>
-				<mesh filename="package://zx120_description/meshes/zx120-arm-cyl2.dae"/>
-			</geometry>
-		</visual>
-		<collision>
-			<origin xyz="0 0 0"/>
-			<geometry>
-				<mesh filename="package://zx120_description/meshes/zx120-arm-cyl2.dae"/>
-			</geometry>
-		</collision>
-		<inertial>
-			<origin xyz="1.686736 -0.001027 -0.000662" rpy="0 0 0"/>
-			<mass value="0.03"/>
-			<inertia ixx="1.0" ixy="0.0" ixz="0.0"
-								iyy="1.0" iyz="0.0"
-											izz="1.0"/>
-		</inertial>
-	</link>
-	<link name="bucket_cylinder_head_link">
-		<visual>
-			<origin xyz="0 0 0"/>
-			<geometry>
-				<mesh filename="package://zx120_description/meshes/zx120-bucket-cyl1.dae"/>
-			</geometry>
-		</visual>
-		<collision>
-			<origin xyz="0 0 0"/>
-			<geometry>
-				<mesh filename="package://zx120_description/meshes/zx120-bucket-cyl1.dae"/>
-			</geometry>
-		</collision>
-		<inertial>
-			<origin xyz="-0.010342 0.000321 -0.639293" rpy="0 0 0"/>
-			<mass value="0.03"/>
-			<inertia ixx="1.0" ixy="0.0" ixz="0.0"
-								iyy="1.0" iyz="0.0"
-											izz="1.0"/>
-		</inertial>
-	</link>
-	<link name="bucket_cylinder_rod_link">
-		<visual>
-			<origin xyz="0 0 0"/>
-			<geometry>
-				<mesh filename="package://zx120_description/meshes/zx120-bucket-cyl2.dae"/>
-			</geometry>
-		</visual>
-		<collision>
-			<origin xyz="0 0 0"/>
-			<geometry>
-				<mesh filename="package://zx120_description/meshes/zx120-bucket-cyl2.dae"/>
-			</geometry>
-		</collision>
-		<inertial>
-			<origin xyz="-0.015456 0.000321 -1.701647" rpy="0 0 0"/>
-			<mass value="0.03"/>
-			<inertia ixx="1.0" ixy="0.0" ixz="0.0"
-								iyy="1.0" iyz="0.0"
-											izz="1.0"/>
-		</inertial>
-	</link>
-	<link name="bucket_b_link">
-		<visual>
-			<origin xyz="0 0 0"/>
-			<geometry>
-				<mesh filename="package://zx120_description/meshes/zx120-p1.dae"/>
-			</geometry>
-		</visual>
-		<collision>
-			<origin xyz="0 0 0"/>
-			<geometry>
-				<mesh filename="package://zx120_description/meshes/zx120-p1.dae"/>
-			</geometry>
-		</collision>
-		<inertial>
-			<origin xyz="0.126203 0.000026 -0.212651" rpy="0 0 0"/>
-			<mass value="0.03"/>
-			<inertia ixx="1.0" ixy="0.0" ixz="0.0"
-								iyy="1.0" iyz="0.0"
-											izz="1.0"/>
-		</inertial>
-	</link>
-	<link name="bucket_a_link">
-		<visual>
-			<origin xyz="0 0 0"/>
-			<geometry>
-				<mesh filename="package://zx120_description/meshes/zx120-p2.dae"/>
-			</geometry>
-		</visual>
-		<collision>
-			<origin xyz="0 0 0"/>
-			<geometry>
-				<mesh filename="package://zx120_description/meshes/zx120-p2.dae"/>
-			</geometry>
-		</collision>
-		<inertial>
-			<origin xyz="0.211197 0.000576 0.111406" rpy="0 0 0"/>
-			<mass value="0.03"/>
-			<inertia ixx="1.0" ixy="0.0" ixz="0.0"
-								iyy="1.0" iyz="0.0"
-											izz="1.0"/>
-		</inertial>
-	</link>
+  <link name="bucket_end_link">
+    <visual>
+      <origin xyz="0 0 0" rpy="0 0 0"/>
+      <geometry>
+        <box size="0.001 0.001 0.001" />
+      </geometry>
+      <material name="red"/>
+    </visual>
+    <inertial>
+      <origin xyz="0 0 0" />
+      <mass value="1.0e-03" />
+      <inertia ixx="1.0e-03" ixy="0.0" ixz="0.0"
+               iyy="1.0e-03" iyz="0.0"
+               izz="1.0e-03" />
+    </inertial>
+  </link>
+  <joint name="bucket_end_joint" type="revolute">
+    <parent link="bucket_link"/>
+    <child link="bucket_end_link"/>
+    <axis xyz="1 0 0"/>
+    <!-- <origin rpy="0 0 0" xyz="0 0 1.23"/> -->
+    <!-- <origin rpy="0 0 0" xyz="-0.723 0 0.995"/> -->
+    <!-- <origin rpy="0 0 0" xyz="-0.85 0 0.889"/> -->
+    <origin rpy="0 ${radians(50)} 0" xyz="0 0 1.23"/>
+    <limit effort="1" lower="-3.14" upper="3.14" velocity="0.5"/>
+  </joint>
 	<transmission name="tran1">
 		<type>transmission_interface/SimpleTransmission</type>
@@ -470,3 +328,13 @@
 		</actuator>
 	</transmission>
+  <transmission name="dummy_trans1">
+    <type>transmission_interface/SimpleTransmission</type>
+      <joint name="bucket_end_joint">
+      <hardwareInterface>hardware_interface/PositionJointInterface</hardwareInterface>
+    </joint>
+    <actuator name="dummy_motor1">
+      <hardwareInterface>hardware_interface/PositionJointInterface</hardwareInterface>
+      <mechanicalReduction>1</mechanicalReduction>
+    </actuator>
+  </transmission>
 </robot>

Commit message: delete mimic joint (hydraulic cylinder)

File: zx120_description/urdf/zx120.xacro (robot description, xacro)
@@ -67,121 +67,4 @@
 		<limit lower="${radians(-70)}" upper="${radians(30)}" effort="500" velocity="6.159937255"/>
 	</joint>
-	<joint name="boom_cylinder_head_joint" type="continuous">
-		<origin xyz="0.556105 -0.164428 0.032962"/>
-		<axis xyz="0 1 0"/>
-		<parent link="body_link"/>
-		<child link="boom_cylinder_head_link"/>
-		<mimic joint="boom_joint" multiplier="${60/70}"/>
-	</joint>
-	<gazebo>
-		<plugin name="boom_cylinder_head_joint_mimic_joint_plugin"
-				filename="libroboticsgroup_upatras_gazebo_mimic_joint_plugin.so">
-			<joint>boom_joint</joint>
-			<mimicJoint>boom_cylinder_head_joint</mimicJoint>
-			<multiplier>${60/70}</multiplier>
-			<offset>0</offset>
-			<robotNamespace>/zx120</robotNamespace>
-		</plugin>
-	</gazebo>
-	<joint name="boom_cylinder_rod_joint" type="prismatic">
-		<origin xyz="0 0 0"/>
-		<axis xyz="0.802033 0 1.847495"/>
-		<parent link="boom_cylinder_head_link"/>
-		<child link="boom_cylinder_rod_link"/>
-		<limit lower="-2" upper="2" effort="500" velocity="6.159937255"/>
-		<mimic joint="boom_joint" multiplier="${0.39/-1.22}"/>
-	</joint>
-	<gazebo>
-		<plugin name="boom_cylinder_rod_joint_mimic_joint_plugin"
-				filename="libroboticsgroup_upatras_gazebo_mimic_joint_plugin.so">
-			<joint>boom_joint</joint>
-			<mimicJoint>boom_cylinder_rod_joint</mimicJoint>
-			<multiplier>${0.39/-1.22}</multiplier>
-			<offset>0</offset>
-			<robotNamespace>/zx120</robotNamespace>
-		</plugin>
-	</gazebo>
-	<joint name="arm_cylinder_head_joint" type="fixed">
-		<origin xyz="2.053030 0 1.991444"/>
-		<axis xyz="0 1 0"/>
-		<parent link="boom_link"/>
-		<child link="arm_cylinder_head_link"/>
-	</joint>
-	<joint name="arm_cylinder_rod_joint" type="prismatic">
-		<origin xyz="0 0 0"/>
-		<axis xyz="2.36471 0 0"/>
-		<parent link="arm_cylinder_head_link"/>
-		<child link="arm_cylinder_rod_link"/>
-		<limit lower="-2" upper="2" effort="500" velocity="6.159937255"/>
-		<mimic joint="arm_joint" multiplier="${0.4/radians(50)}"/>
-	</joint>
-	<gazebo>
-		<plugin name="arm_cylinder_rod_joint_mimic_joint_plugin"
-				filename="libroboticsgroup_upatras_gazebo_mimic_joint_plugin.so">
-			<joint>arm_joint</joint>
-			<mimicJoint>arm_cylinder_rod_joint</mimicJoint>
-			<multiplier>${0.4/radians(50)}</multiplier>
-			<offset>0</offset>
-			<robotNamespace>/zx120</robotNamespace>
-		</plugin>
-	</gazebo>
-	<joint name="bucket_cylinder_head_joint" type="fixed">
-		<origin xyz="0.605825 0 -0.364793"/>
-		<axis xyz="0 1 0"/>
-		<parent link="arm_link"/>
-		<child link="bucket_cylinder_head_link"/>
-	</joint>
-	<joint name="bucket_cylinder_rod_joint" type="prismatic">
-		<origin xyz="0 0 0"/>
-		<axis xyz="-0.021529 0 -2.207579"/>
-		<parent link="bucket_cylinder_head_link"/>
-		<child link="bucket_cylinder_rod_link"/>
-		<limit lower="-2" upper="2" effort="500" velocity="6.159937255"/>
-		<mimic joint="bucket_joint" multiplier="${-0.9/-2.79}"/>
-	</joint>
-	<gazebo>
-		<plugin name="bucket_cylinder_rod_joint_mimic_joint_plugin"
-				filename="libroboticsgroup_upatras_gazebo_mimic_joint_plugin.so">
-			<joint>bucket_joint</joint>
-			<mimicJoint>bucket_cylinder_rod_joint</mimicJoint>
-			<multiplier>${-0.9/-2.79}</multiplier>
-			<offset>0</offset>
-			<robotNamespace>/zx120</robotNamespace>
-		</plugin>
-	</gazebo>
-	<joint name="bucket_b_joint" type="continuous">
-		<origin xyz="0.330489 0 -2.150643"/>
-		<axis xyz="0 1 0"/>
-		<parent link="arm_link"/>
-		<child link="bucket_b_link"/>
-		<mimic joint="bucket_joint" multiplier="${120/160}"/>
-	</joint>
-	<gazebo>
-		<plugin name="bucket_b_joint_mimic_joint_plugin"
-				filename="libroboticsgroup_upatras_gazebo_mimic_joint_plugin.so">
-			<joint>bucket_joint</joint>
-			<mimicJoint>bucket_b_joint</mimicJoint>
-			<multiplier>${120/160}</multiplier>
-			<offset>0</offset>
-			<robotNamespace>/zx120</robotNamespace>
-		</plugin>
-	</gazebo>
-	<joint name="bucket_a_joint" type="continuous">
-		<origin xyz="-0.182145 0 -0.315076"/>
-		<axis xyz="0 1 0"/>
-		<parent link="bucket_link"/>
-		<child link="bucket_a_link"/>
-		<mimic joint="bucket_joint" multiplier="${-92/160}"/>
-	</joint>
-	<gazebo>
-		<plugin name="bucket_a_joint_mimic_joint_plugin"
-				filename="libroboticsgroup_upatras_gazebo_mimic_joint_plugin.so">
-			<joint>bucket_joint</joint>
-			<mimicJoint>bucket_a_joint</mimicJoint>
-			<multiplier>${-92/160}</multiplier>
-			<offset>0</offset>
-			<robotNamespace>/zx120</robotNamespace>
-		</plugin>
-	</gazebo>
 	<link name="boom_link">
 		<visual>
